Commit message: FAILED AT GAZEBO SIMULATION. tried to add IMU to the urdf, but unsuccessful. will return once design has been finalised

File: ros2_ws/install/my_package/share/my_package/description/truck_robot.urdf.xacro (robot description, xacro)
@@ -1,4 +1,5 @@
 <?xml version="1.0"?>
 <robot xmlns:xacro="http://www.ros.org/wiki/xacro" name="truck_robot">
+  <!-- Material definitions for RViz2 -->
   <material name="gray">
     <color rgba="0.5 0.5 0.5 1"/>
@@ -13,8 +14,7 @@
     <color rgba="0.1 0.1 0.1 1"/>
   </material>
-  <material name="green">
-    <color rgba="0.1 0.8 0.1 1"/>
-  </material>
+  <!-- Define xacro properties for easy customization -->
   <xacro:property name="PI" value="3.14159265359"/>
+  <!-- Truck dimensions -->
   <xacro:property name="chassis_length" value="1.2"/>
   <xacro:property name="chassis_width" value="0.5"/>
@@ -25,5 +25,6 @@
   <xacro:property name="cabin_height" value="0.35"/>
   <xacro:property name="cabin_mass" value="5.0"/>
-  <xacro:property name="wheel_radius" value="0.078"/>
+  <!-- Wheel properties -->
+  <xacro:property name="wheel_radius" value="0.1"/>
   <xacro:property name="wheel_width" value="0.08"/>
   <xacro:property name="wheel_mass" value="1.0"/>
@@ -31,14 +32,14 @@
   <xacro:property name="wheel_offset_y" value="0.3"/>
   <xacro:property name="wheel_offset_z" value="0.0"/>
+  <!-- LIDAR properties -->
   <xacro:property name="lidar_radius" value="0.05"/>
   <xacro:property name="lidar_height" value="0.07"/>
   <xacro:property name="lidar_mass" value="0.3"/>
+  <!-- Camera properties -->
   <xacro:property name="camera_size" value="0.05"/>
   <xacro:property name="camera_mass" value="0.1"/>
-  <xacro:property name="imu_size" value="0.02"/>
-  <xacro:property name="imu_mass" value="0.015"/>
+  <!-- Macro for inertial properties of a box -->
   <xacro:macro name="box_inertia" params="mass length width height">
     <inertial>
-      <origin xyz="0 0 0" rpy="0 0 0"/>
       <mass value="${mass}"/>
       <inertia ixx="${(1/12) * mass * (width*width + height*height)}" ixy="0.0" ixz="0.0"
@@ -47,7 +48,7 @@
     </inertial>
   </xacro:macro>
+  <!-- Macro for inertial properties of a cylinder -->
   <xacro:macro name="cylinder_inertia" params="mass radius height">
     <inertial>
-      <origin xyz="0 0 0" rpy="0 0 0"/>
       <mass value="${mass}"/>
       <inertia ixx="${(1/12) * mass * (3*radius*radius + height*height)}" ixy="0.0" ixz="0.0"
@@ -56,4 +57,5 @@
     </inertial>
   </xacro:macro>
+  <!-- Macro for wheels -->
   <xacro:macro name="wheel" params="prefix reflect_y reflect_x">
     <link name="${prefix}_wheel">
@@ -63,5 +65,7 @@
           <cylinder radius="${wheel_radius}" length="${wheel_width}"/>
         </geometry>
-        <material name="black"/>
+        <material name="black">
+          <color rgba="0.1 0.1 0.1 1"/>
+        </material>
       </visual>
       <collision>
@@ -80,5 +84,7 @@
     </joint>
   </xacro:macro>
+  <!-- Base footprint (for navigation) -->
   <link name="base_footprint"/>
+  <!-- Base link (chassis) -->
   <link name="base_link">
     <visual>
@@ -87,5 +93,7 @@
         <box size="${chassis_length} ${chassis_width} ${chassis_height}"/>
       </geometry>
-      <material name="gray"/>
+      <material name="gray">
+        <color rgba="0.5 0.5 0.5 1"/>
+      </material>
     </visual>
     <collision>
@@ -97,4 +105,5 @@
     <xacro:box_inertia mass="${chassis_mass}" length="${chassis_length}" width="${chassis_width}" height="${chassis_height}"/>
   </link>
+  <!-- Joint connecting footprint to base_link -->
   <joint name="base_joint" type="fixed">
     <parent link="base_footprint"/>
@@ -102,4 +111,5 @@
     <origin xyz="0 0 ${wheel_radius}" rpy="0 0 0"/>
   </joint>
+  <!-- Cabin link -->
   <link name="cabin_link">
     <visual>
@@ -108,5 +118,7 @@
         <box size="${cabin_length} ${cabin_width} ${cabin_height}"/>
       </geometry>
-      <material name="blue"/>
+      <material name="blue">
+        <color rgba="0.2 0.4 0.8 1"/>
+      </material>
     </visual>
     <collision>
@@ -118,4 +130,5 @@
     <xacro:box_inertia mass="${cabin_mass}" length="${cabin_length}" width="${cabin_width}" height="${cabin_height}"/>
   </link>
+  <!-- Joint connecting cabin to chassis -->
   <joint name="cabin_joint" type="fixed">
     <parent link="base_link"/>
@@ -123,12 +136,17 @@
     <origin xyz="${chassis_length/2 - cabin_length/2} 0 ${chassis_height}" rpy="0 0 0"/>
   </joint>
+  <!-- LIDAR link -->
   <link name="lidar_link">
     <visual>
+      <origin xyz="0 0 0" rpy="0 0 0"/>
       <geometry>
         <cylinder radius="${lidar_radius}" length="${lidar_height}"/>
       </geometry>
-      <material name="red"/>
-    </visual>
-    <collision>
+      <material name="red">
+        <color rgba="0.8 0.1 0.1 1"/>
+      </material>
+    </visual>
+    <collision>
+      <origin xyz="0 0 0" rpy="0 0 0"/>
       <geometry>
         <cylinder radius="${lidar_radius}" length="${lidar_height}"/>
@@ -137,4 +155,5 @@
     <xacro:cylinder_inertia mass="${lidar_mass}" radius="${lidar_radius}" height="${lidar_height}"/>
   </link>
+  <!-- Joint connecting LIDAR to cabin top -->
   <joint name="lidar_joint" type="fixed">
     <parent link="cabin_link"/>
@@ -142,12 +161,17 @@
     <origin xyz="0 0 ${cabin_height + lidar_height/2}" rpy="0 0 0"/>
   </joint>
+  <!-- Camera link -->
   <link name="camera">
     <visual>
+      <origin xyz="0 0 0" rpy="0 0 0"/>
       <geometry>
         <box size="${camera_size} ${camera_size} ${camera_size}"/>
       </geometry>
-      <material name="black"/>
-    </visual>
-    <collision>
+      <material name="black">
+        <color rgba="0.1 0.1 0.1 1"/>
+      </material>
+    </visual>
+    <collision>
+      <origin xyz="0 0 0" rpy="0 0 0"/>
       <geometry>
         <box size="${camera_size} ${camera_size} ${camera_size}"/>
@@ -156,4 +180,5 @@
     <xacro:box_inertia mass="${camera_mass}" length="${camera_size}" width="${camera_size}" height="${camera_size}"/>
   </link>
+  <!-- Joint connecting camera to cabin front -->
   <joint name="camera_joint" type="fixed">
     <parent link="cabin_link"/>
@@ -161,65 +186,23 @@
     <origin xyz="${cabin_length/2} 0 ${cabin_height/2}" rpy="0 0 0"/>
   </joint>
-  <link name="imu_link">
-    <visual>
-      <geometry>
-        <box size="${imu_size} ${imu_size} ${imu_size}"/>
-      </geometry>
-      <material name="green"/>
-    </visual>
-    <collision>
-      <geometry>
-        <box size="${imu_size} ${imu_size} ${imu_size}"/>
-      </geometry>
-    </collision>
-    <xacro:box_inertia mass="${imu_mass}" length="${imu_size}" width="${imu_size}" height="${imu_size}"/>
-  </link>
-  <joint name="imu_joint" type="fixed">
-    <parent link="base_link"/>
-    <child link="imu_link"/>
-    <origin xyz="0 0 ${chassis_height}" rpy="0 0 0"/>
-  </joint>
+  <!-- Instantiate wheels -->
   <xacro:wheel prefix="front_left" reflect_y="1" reflect_x="1"/>
   <xacro:wheel prefix="front_right" reflect_y="-1" reflect_x="1"/>
   <xacro:wheel prefix="rear_left" reflect_y="1" reflect_x="-1"/>
   <xacro:wheel prefix="rear_right" reflect_y="-1" reflect_x="-1"/>
-  <gazebo reference="front_left_wheel">
-    <mu1>0.5</mu1>
-    <mu2>0.5</mu2>
-  </gazebo>
-  <gazebo reference="front_right_wheel">
-    <mu1>0.5</mu1>
-    <mu2>0.5</mu2>
-  </gazebo>
-  <gazebo reference="rear_left_wheel">
-    <mu1>0.5</mu1>
-    <mu2>0.5</mu2>
-  </gazebo>
-  <gazebo reference="rear_right_wheel">
-    <mu1>0.5</mu1>
-    <mu2>0.5</mu2>
-  </gazebo>
-  <gazebo>
-    <plugin filename="libignition-gazebo-diff-drive-system.so" name="ignition::gazebo::systems::DiffDrive">
-      <left_joint>front_left_wheel_joint</left_joint>
-      <left_joint>rear_left_wheel_joint</left_joint>
-      <right_joint>front_right_wheel_joint</right_joint>
-      <right_joint>rear_right_wheel_joint</right_joint>
-      <wheel_separation>${wheel_offset_y * 2}</wheel_separation>
-      <wheel_radius>${wheel_radius}</wheel_radius>
-      <odometry_source>world</odometry_source>
-      <topic>cmd_vel</topic>
-      <odom_topic>odom</odom_topic>
-      <tf_topic>/tf</tf_topic>
-      <frame_id>odom</frame_id>
-      <child_frame_id>base_footprint</child_frame_id>
-    </plugin>
+  <!-- Gazebo-specific elements (optional but recommended) -->
+  <gazebo reference="base_link">
+    <material>Gazebo/Grey</material>
+  </gazebo>
+  <gazebo reference="cabin_link">
+    <material>Gazebo/Blue</material>
   </gazebo>
   <gazebo reference="lidar_link">
-    <sensor name="lidar_sensor" type="gpu_lidar">
-      <topic>scan</topic>
-      <update_rate>10.0</update_rate>
-      <gz_frame_id>lidar_link</gz_frame_id>
-      <lidar>
+    <material>Gazebo/Red</material>
+    <sensor type="ray" name="lidar_sensor">
+      <pose>0 0 0 0 0 0</pose>
+      <visualize>true</visualize>
+      <update_rate>10</update_rate>
+      <ray>
         <scan>
           <horizontal>
@@ -232,34 +215,42 @@
         <range>
           <min>0.2</min>
-          <max>5.0</max>
+          <max>30.0</max>
           <resolution>0.01</resolution>
         </range>
-      </lidar>
-      <always_on>true</always_on>
-      <visualize>true</visualize>
+        <noise>
+          <type>gaussian</type>
+          <mean>0.0</mean>
+          <stddev>0.01</stddev>
+        </noise>
+      </ray>
+      <plugin name="gazebo_ros_lidar" filename="libgazebo_ros_ray_sensor.so">
+        <ros>
+          <namespace>/truck_robot</namespace>
+          <remapping>~/out:=scan</remapping>
+        </ros>
+        <output_type>sensor_msgs/LaserScan</output_type>
+        <frame_name>lidar_link</frame_name>
+      </plugin>
     </sensor>
   </gazebo>
-  <!-- <gazebo reference="imu_link">
-    <sensor name="imu_sensor" type="imu">
-      <topic>imu</topic>
-      <update_rate>100</update_rate>
-      <gz_frame_id>imu_link</gz_frame_id>
-      <always_on>true</always_on>
-    </sensor>
-  </gazebo> -->
   <gazebo>
-    <plugin filename="libignition-gazebo-sensors-system.so" name="ignition::gazebo::systems::Sensors">
-      <render_engine>ogre2</render_engine>
+    <plugin name="gazebo_ros_diff_drive" filename="libgazebo_ros_diff_drive.so">
+      <update_rate>50</update_rate>
+      <left_joint>front_left_wheel_joint</left_joint>
+      <left_joint>rear_left_wheel_joint</left_joint>
+      <right_joint>front_right_wheel_joint</right_joint>
+      <right_joint>rear_right_wheel_joint</right_joint>
+      <wheel_separation>${wheel_offset_y * 2}</wheel_separation>
+      <wheel_diameter>${wheel_radius * 2}</wheel_diameter>
+      <max_wheel_torque>20</max_wheel_torque>
+      <max_wheel_acceleration>1.0</max_wheel_acceleration>
+      <command_topic>cmd_vel</command_topic>
+      <publish_odom>true</publish_odom>
+      <publish_odom_tf>true</publish_odom_tf>
+      <publish_wheel_tf>true</publish_wheel_tf>
+      <odometry_topic>odom</odometry_topic>
+      <odometry_frame>odom</odometry_frame>
+      <robot_base_frame>base_footprint</robot_base_frame>
     </plugin>
   </gazebo>
-  <gazebo>
-    <plugin filename="libignition-gazebo-joint-state-publisher-system.so" name="ignition::gazebo::systems::JointStatePublisher"/>
-  </gazebo>
-  <gazebo reference="base_link">
-    <sensor name="imu_sensor" type="imu">
-      <topic>imu</topic>
-      <update_rate>100</update_rate>
-      <always_on>true</always_on>
-    </sensor>
-  </gazebo>
 </robot>

File: ros2_ws/src/my_package/description/truck_robot_ign.urdf copy.xacro (robot description, xacro)
@@ -1,4 +1,5 @@
 <?xml version="1.0"?>
 <robot xmlns:xacro="http://www.ros.org/wiki/xacro" name="truck_robot">
+  <!-- Material definitions for RViz2 -->
   <material name="gray">
     <color rgba="0.5 0.5 0.5 1"/>
@@ -13,8 +14,7 @@
     <color rgba="0.1 0.1 0.1 1"/>
   </material>
-  <material name="green">
-    <color rgba="0.1 0.8 0.1 1"/>
-  </material>
+  <!-- Define xacro properties for easy customization -->
   <xacro:property name="PI" value="3.14159265359"/>
+  <!-- Truck dimensions -->
   <xacro:property name="chassis_length" value="1.2"/>
   <xacro:property name="chassis_width" value="0.5"/>
@@ -25,4 +25,5 @@
   <xacro:property name="cabin_height" value="0.35"/>
   <xacro:property name="cabin_mass" value="5.0"/>
+  <!-- Wheel properties -->
   <xacro:property name="wheel_radius" value="0.078"/>
   <xacro:property name="wheel_width" value="0.08"/>
@@ -31,11 +32,12 @@
   <xacro:property name="wheel_offset_y" value="0.3"/>
   <xacro:property name="wheel_offset_z" value="0.0"/>
+  <!-- LIDAR properties -->
   <xacro:property name="lidar_radius" value="0.05"/>
   <xacro:property name="lidar_height" value="0.07"/>
   <xacro:property name="lidar_mass" value="0.3"/>
+  <!-- Camera properties -->
   <xacro:property name="camera_size" value="0.05"/>
   <xacro:property name="camera_mass" value="0.1"/>
-  <xacro:property name="imu_size" value="0.02"/>
-  <xacro:property name="imu_mass" value="0.015"/>
+  <!-- Macro for inertial properties of a box -->
   <xacro:macro name="box_inertia" params="mass length width height">
     <inertial>
@@ -47,4 +49,5 @@
     </inertial>
   </xacro:macro>
+  <!-- Macro for inertial properties of a cylinder -->
   <xacro:macro name="cylinder_inertia" params="mass radius height">
     <inertial>
@@ -56,4 +59,5 @@
     </inertial>
   </xacro:macro>
+  <!-- Macro for wheels -->
   <xacro:macro name="wheel" params="prefix reflect_y reflect_x">
     <link name="${prefix}_wheel">
@@ -63,5 +67,7 @@
           <cylinder radius="${wheel_radius}" length="${wheel_width}"/>
         </geometry>
-        <material name="black"/>
+        <material name="black">
+          <color rgba="0.1 0.1 0.1 1"/>
+        </material>
       </visual>
       <collision>
@@ -80,5 +86,7 @@
     </joint>
   </xacro:macro>
+  <!-- Base footprint (for navigation) -->
   <link name="base_footprint"/>
+  <!-- Base link (chassis) -->
   <link name="base_link">
     <visual>
@@ -87,5 +95,7 @@
         <box size="${chassis_length} ${chassis_width} ${chassis_height}"/>
       </geometry>
-      <material name="gray"/>
+      <material name="gray">
+        <color rgba="0.5 0.5 0.5 1"/>
+      </material>
     </visual>
     <collision>
@@ -97,4 +107,5 @@
     <xacro:box_inertia mass="${chassis_mass}" length="${chassis_length}" width="${chassis_width}" height="${chassis_height}"/>
   </link>
+  <!-- Joint connecting footprint to base_link -->
   <joint name="base_joint" type="fixed">
     <parent link="base_footprint"/>
@@ -102,4 +113,5 @@
     <origin xyz="0 0 ${wheel_radius}" rpy="0 0 0"/>
   </joint>
+  <!-- Cabin link -->
   <link name="cabin_link">
     <visual>
@@ -108,5 +120,7 @@
         <box size="${cabin_length} ${cabin_width} ${cabin_height}"/>
       </geometry>
-      <material name="blue"/>
+      <material name="blue">
+        <color rgba="0.2 0.4 0.8 1"/>
+      </material>
     </visual>
     <collision>
@@ -118,4 +132,5 @@
     <xacro:box_inertia mass="${cabin_mass}" length="${cabin_length}" width="${cabin_width}" height="${cabin_height}"/>
   </link>
+  <!-- Joint connecting cabin to chassis -->
   <joint name="cabin_joint" type="fixed">
     <parent link="base_link"/>
@@ -123,12 +138,17 @@
     <origin xyz="${chassis_length/2 - cabin_length/2} 0 ${chassis_height}" rpy="0 0 0"/>
   </joint>
+  <!-- LIDAR link -->
   <link name="lidar_link">
     <visual>
+      <origin xyz="0 0 0" rpy="0 0 0"/>
       <geometry>
         <cylinder radius="${lidar_radius}" length="${lidar_height}"/>
       </geometry>
-      <material name="red"/>
-    </visual>
-    <collision>
+      <material name="red">
+        <color rgba="0.8 0.1 0.1 1"/>
+      </material>
+    </visual>
+    <collision>
+      <origin xyz="0 0 0" rpy="0 0 0"/>
       <geometry>
         <cylinder radius="${lidar_radius}" length="${lidar_height}"/>
@@ -137,4 +157,5 @@
     <xacro:cylinder_inertia mass="${lidar_mass}" radius="${lidar_radius}" height="${lidar_height}"/>
   </link>
+  <!-- Joint connecting LIDAR to cabin top -->
   <joint name="lidar_joint" type="fixed">
     <parent link="cabin_link"/>
@@ -142,12 +163,17 @@
     <origin xyz="0 0 ${cabin_height + lidar_height/2}" rpy="0 0 0"/>
   </joint>
+  <!-- Camera link -->
   <link name="camera">
     <visual>
+      <origin xyz="0 0 0" rpy="0 0 0"/>
       <geometry>
         <box size="${camera_size} ${camera_size} ${camera_size}"/>
       </geometry>
-      <material name="black"/>
-    </visual>
-    <collision>
+      <material name="black">
+        <color rgba="0.1 0.1 0.1 1"/>
+      </material>
+    </visual>
+    <collision>
+      <origin xyz="0 0 0" rpy="0 0 0"/>
       <geometry>
         <box size="${camera_size} ${camera_size} ${camera_size}"/>
@@ -156,4 +182,5 @@
     <xacro:box_inertia mass="${camera_mass}" length="${camera_size}" width="${camera_size}" height="${camera_size}"/>
   </link>
+  <!-- Joint connecting camera to cabin front -->
   <joint name="camera_joint" type="fixed">
     <parent link="cabin_link"/>
@@ -161,44 +188,40 @@
     <origin xyz="${cabin_length/2} 0 ${cabin_height/2}" rpy="0 0 0"/>
   </joint>
-  <link name="imu_link">
-    <visual>
-      <geometry>
-        <box size="${imu_size} ${imu_size} ${imu_size}"/>
-      </geometry>
-      <material name="green"/>
-    </visual>
-    <collision>
-      <geometry>
-        <box size="${imu_size} ${imu_size} ${imu_size}"/>
-      </geometry>
-    </collision>
-    <xacro:box_inertia mass="${imu_mass}" length="${imu_size}" width="${imu_size}" height="${imu_size}"/>
-  </link>
-  <joint name="imu_joint" type="fixed">
-    <parent link="base_link"/>
-    <child link="imu_link"/>
-    <origin xyz="0 0 ${chassis_height}" rpy="0 0 0"/>
-  </joint>
-  <xacro:wheel prefix="front_left" reflect_y="1" reflect_x="1"/>
-  <xacro:wheel prefix="front_right" reflect_y="-1" reflect_x="1"/>
-  <xacro:wheel prefix="rear_left" reflect_y="1" reflect_x="-1"/>
-  <xacro:wheel prefix="rear_right" reflect_y="-1" reflect_x="-1"/>
-  <gazebo reference="front_left_wheel">
-    <mu1>0.5</mu1>
-    <mu2>0.5</mu2>
-  </gazebo>
-  <gazebo reference="front_right_wheel">
-    <mu1>0.5</mu1>
-    <mu2>0.5</mu2>
-  </gazebo>
-  <gazebo reference="rear_left_wheel">
-    <mu1>0.5</mu1>
-    <mu2>0.5</mu2>
-  </gazebo>
-  <gazebo reference="rear_right_wheel">
-    <mu1>0.5</mu1>
-    <mu2>0.5</mu2>
-  </gazebo>
+  <!-- Instantiate wheels -->
+<xacro:wheel prefix="front_left" reflect_y="1" reflect_x="1"/>
+<xacro:wheel prefix="front_right" reflect_y="-1" reflect_x="1"/>
+<xacro:wheel prefix="rear_left" reflect_y="1" reflect_x="-1"/>
+<xacro:wheel prefix="rear_right" reflect_y="-1" reflect_x="-1"/>
+<!-- ADD THESE WHEEL FRICTION PARAMETERS -->
+<gazebo reference="front_left_wheel">
+  <mu1>1.0</mu1>
+  <mu2>1.0</mu2>
+  <kp>10000000.0</kp>
+  <kd>1.0</kd>
+  <minDepth>0.001</minDepth>
+</gazebo>
+<gazebo reference="front_right_wheel">
+  <mu1>1.0</mu1>
+  <mu2>1.0</mu2>
+  <kp>10000000.0</kp>
+  <kd>1.0</kd>
+  <minDepth>0.001</minDepth>
+</gazebo>
+<gazebo reference="rear_left_wheel">
+  <mu1>1.0</mu1>
+  <mu2>1.0</mu2>
+  <kp>10000000.0</kp>
+  <kd>1.0</kd>
+  <minDepth>0.001</minDepth>
+</gazebo>
+<gazebo reference="rear_right_wheel">
+  <mu1>1.0</mu1>
+  <mu2>1.0</mu2>
+  <kp>10000000.0</kp>
+  <kd>1.0</kd>
+  <minDepth>0.001</minDepth>
+</gazebo>
   <gazebo>
+    <!-- Differential Drive Controller for Ignition Gazebo -->
     <plugin filename="libignition-gazebo-diff-drive-system.so" name="ignition::gazebo::systems::DiffDrive">
       <left_joint>front_left_wheel_joint</left_joint>
@@ -208,5 +231,7 @@
       <wheel_separation>${wheel_offset_y * 2}</wheel_separation>
       <wheel_radius>${wheel_radius}</wheel_radius>
+      <!-- ADD THIS LINE: Use perfect physics-based odometry -->
       <odometry_source>world</odometry_source>
+      <odom_publish_frequency>50</odom_publish_frequency>
       <topic>cmd_vel</topic>
       <odom_topic>odom</odom_topic>
@@ -216,4 +241,5 @@
     </plugin>
   </gazebo>
+  <!-- LIDAR sensor for Ignition Gazebo -->
   <gazebo reference="lidar_link">
     <sensor name="lidar_sensor" type="gpu_lidar">
@@ -240,12 +266,5 @@
     </sensor>
   </gazebo>
-  <!-- <gazebo reference="imu_link">
-    <sensor name="imu_sensor" type="imu">
-      <topic>imu</topic>
-      <update_rate>100</update_rate>
-      <gz_frame_id>imu_link</gz_frame_id>
-      <always_on>true</always_on>
-    </sensor>
-  </gazebo> -->
+  <!-- Sensors system plugin -->
   <gazebo>
     <plugin filename="libignition-gazebo-sensors-system.so" name="ignition::gazebo::systems::Sensors">
@@ -253,13 +272,13 @@
     </plugin>
   </gazebo>
+  <!-- Joint State Publisher plugin -->
   <gazebo>
-    <plugin filename="libignition-gazebo-joint-state-publisher-system.so" name="ignition::gazebo::systems::JointStatePublisher"/>
-  </gazebo>
-  <gazebo reference="base_link">
-    <sensor name="imu_sensor" type="imu">
-      <topic>imu</topic>
-      <update_rate>100</update_rate>
-      <always_on>true</always_on>
-    </sensor>
+  <plugin filename="libignition-gazebo-joint-state-publisher-system.so"
+          name="ignition::gazebo::systems::JointStatePublisher">
+    <joint_name>front_left_wheel_joint</joint_name>
+    <joint_name>front_right_wheel_joint</joint_name>
+    <joint_name>rear_left_wheel_joint</joint_name>
+    <joint_name>rear_right_wheel_joint</joint_name>
+  </plugin>
   </gazebo>
 </robot>
